Commit message: Fine tuned simple geometry

File: robots/so_arm_description/urdf/so101_simple_collision.urdf (robot description, URDF)
Before this commit: robot so101_simple_collision, 8 links, 7 joints
Links:
- link base_link: geometry collision box size=0.02 0.035 0.02; collision box size=0.038 0.05 0.07
- link gripper_link: geometry collision box size=0.012 0.015 0.05; collision box size=0.02 0.026 0.04
- link lower_arm_link: geometry collision box size=0.03 0.036 0.07; collision box size=0.110 0.025 0.07
- link moving_jaw_so101_v1_link: geometry collision box size=0.011 0.032 0.018; collision box size=0.02 0.03 0.02
- link shoulder_link: geometry collision box size=0.025 0.040 0.04; collision box size=0.04 0.055 0.025
- link upper_arm_link: geometry collision box size=0.12 0.026 0.07; visual mesh filename=package://example-robot-data/robots/so_arm_description/mesh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
- link wrist_link: geometry collision box size=0.024 0.034 0.062; collision box size=0.036 0.033 0.058
